Commit message: Modified the robot apparance and made driving toward the ball mode accurate

File: src/my_robot/urdf/my_robot.xacro (robot description, xacro)
@@ -22,5 +22,6 @@
             <origin xyz="0 0 0" rpy=" 0 0 0"/>
             <geometry>
-                <box size=".4 .2 .1"/>
+                <!-- <box size=".4 .2 .1"/> -->
+                <cylinder length=".1" radius=".2" />
             </geometry>
         </collision>
@@ -28,5 +29,5 @@
             <origin xyz="0 0 0" rpy=" 0 0 0"/>
             <geometry>
-                <box size=".4 .2 .1"/>
+                <cylinder length=".1" radius=".2" />
             </geometry>
         </visual>
@@ -172,5 +173,6 @@
     </joint>
     <joint type="fixed" name="hokuyo_joint">
-        <origin xyz="0.15 0 0.1" rpy="0 0 0"/>
+        <!-- <origin xyz="0.15 0 0.1" rpy="0 0 0"/> -->
+        <origin xyz="0 0 0.1" rpy="0 0 0"/>
         <child link="hokuyo"/>
         <parent link="chassis"/>
